File: Circuit/ControlTester/ControlTester.kicad_pcb (KiCad board)
At the start: 2 copper layers, 17.8 x 50.8 mm, 13 parts, among them J1 Power, J2 Signal, J3 NO G NC

Commit message: [Circuit] Use a single 12V power for control module
Parts:
- J1: footprint Connector_PinHeader_2.54mm:PinHeader_1x03_P2.54mm_Vertical -> Connector_PinHeader_2.54mm:PinHeader_1x02_P2.54mm_Vertical
- J3: value NO G NC -> 12V NO G
- moved R3 12.7 mm to (81.3, 73.7), turned to 270 degrees
- moved R6 7.62 mm to (83.8, 94.0)
- moved D2 7.18 mm to (91.4, 91.4), turned to 90 degrees
- moved J3 5.08 mm to (81.3, 86.4)
- moved R4 2.54 mm to (83.8, 81.3), turned to 0 degrees
- turned D1 to 90 degrees
Connections:
- D1 pad 1: GND -> Net-(D1-Pad1)
- D2 pad 1: GND -> Net-(D2-Pad1)
- D2 pad 2: Net-(D2-Pad2) -> Net-(D1-Pad1)
- J3 pad 2: GND -> Net-(D1-Pad1)
- R3 pad 1: Net-(R3-Pad1) -> +12V
- R4 pad 2: -12V -> Net-(R4-Pad2)
- R6 pad 2: Net-(D2-Pad2) -> Net-(D2-Pad1)
- RV2 pad 1: GND -> Net-(R4-Pad2)
- RV2 pad 3: Net-(R3-Pad1) -> GND
Routing:
- net GND: track 49.3 -> 23.9 mm
- net Net-(R4-Pad2): track 0.00 -> 12.3 mm
- net Net-(D1-Pad1): track 0.00 -> 12.3 mm
- net +12V: track 2.54 -> 11.2 mm
- net Net-(R3-Pad1): track 6.13 -> 0.00 mm
- net Net-(D2-Pad2): track 6.13 -> 0.00 mm
- net Net-(J3-Pad1): track 6.13 -> 2.54 mm
- net Net-(D2-Pad1): track 0.00 -> 2.54 mm
- net Net-(J3-Pad3): track 6.13 -> 3.59 mm
- net -12V: track 2.54 -> 0.00 mm
Other:
- board size 17.8 x 50.8 mm -> 17.8 x 43.2 mm
