File: Circuit/CapacitorBank/Transformer.kicad_pcb (KiCad board)
At the start: 2 copper layers, 25.4 x 61 mm, 10 parts, among them J1 AC Power In, J2 To Capacitors, T1 6:200

Commit message: [Circuit] Add PCB design for starter
Parts:
- moved J1 5.08 mm to (132.1, 76.2), turned to 90 degrees
Connections:
- J1 pad 1: /ACPowerIn+ -> /ACPowerIn-
- J1 pad 2: /ACPowerIn- -> /ACPowerIn+
Changed lines of the file:
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@@
   )
   (module TerminalBlock:TerminalBlock_bornier-2_P5.08mm (layer F.Cu)
-    (at 132.08 71.12 270)
+    (at 132.08 76.2 90)
     (descr "simple 2-pin terminal block, pitch 5.08mm, revamped version of bornier2")
     (tags "terminal block bornier2")
@@
       (effects (font (size 1 1) (thickness 0.15)))
     )
-    (pad 2 thru_hole circle (at 5.08 0 270) (size 3 3) (drill 1.52) (layers *.Cu *.Mask)
+    (pad 2 thru_hole circle (at 5.08 0 90) (size 3 3) (drill 1.52) (layers *.Cu *.Mask)
+      (net 8 /ACPowerIn+))
+    (pad 1 thru_hole rect (at 0 0 90) (size 3 3) (drill 1.52) (layers *.Cu *.Mask)
       (net 7 /ACPowerIn-))
-    (pad 1 thru_hole rect (at 0 0 270) (size 3 3) (drill 1.52) (layers *.Cu *.Mask)
-      (net 8 /ACPowerIn+))
     (model ${KISYS3DMOD}/TerminalBlock.3dshapes/TerminalBlock_bornier-2_P5.08mm.wrl
       (offset (xyz 2.539999961853027 0 0))
@@
     (pad 2 thru_hole circle (at 5 0 270) (size 2 2) (drill 0.9) (layers *.Cu *.Mask))
     (pad 1 thru_hole rect (at 0 0 270) (size 2 2) (drill 0.9) (layers *.Cu *.Mask))
-    (model ${KISYS3DMOD}/Transformer_THT.3dshapes/Transformer_Breve_TEZ-22x24.wrl
-      (at (xyz 0 0 0))
-      (scale (xyz 1 1 1))
-      (rotate (xyz 0 0 0))
-    )
   )
   (module Capacitor_THT:C_Disc_D4.7mm_W2.5mm_P5.00mm (layer F.Cu)
