File: Circuit/CapacitorBank/VoltageSensingTester.kicad_pcb (KiCad board)
At the start: 2 copper layers, 25.4 x 25.4 mm, 9 parts, among them J1 Conn_01x02_Male, J2 Conn_01x02_Male

Commit message: [Circuit] Update the control test module to use on the new control module
Parts:
- BT1, BT2: value Battery -> 12V Battery
Changed lines of the file:
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@@
     (solder_mask_min_width 0.25)
     (aux_axis_origin 0 0)
-    (visible_elements FFFFFF7F)
+    (visible_elements 7FFFFFFF)
     (pcbplotparams
       (layerselection 0x010fc_ffffffff)
@@
       (effects (font (size 1 1) (thickness 0.15)))
     )
-    (fp_text value Battery (at 0 4.87 90) (layer F.Fab)
+    (fp_text value "12V Battery" (at 0 4.87 90) (layer F.Fab)
       (effects (font (size 1 1) (thickness 0.15)))
     )
@@
       (effects (font (size 1 1) (thickness 0.15)))
     )
-    (fp_text value Battery (at 0 4.87 90) (layer F.Fab)
+    (fp_text value "12V Battery" (at 0 4.87 90) (layer F.Fab)
       (effects (font (size 1 1) (thickness 0.15)))
     )

Commit message: [Circuit] Optimize the interface between capacitor bank modules and voltage sensing module
Parts:
- R1: value 10K -> 47K
Changed lines of the file:
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@@
       (effects (font (size 1 1) (thickness 0.15)))
     )
-    (fp_text value 10K (at 3.81 2.37 90) (layer F.Fab)
+    (fp_text value 47K (at 3.81 2.37 90) (layer F.Fab)
       (effects (font (size 1 1) (thickness 0.15)))
     )
