File: Circuit/PropellantInjector/PropellantInjector.kicad_pcb (KiCad board)
At the start: 2 copper layers, 27.9 x 15.2 mm, 3 parts, among them J1 Injector Power, M1 Motor_DC

Commit message: [Circuit] Upgrade to KiCad 6 format
Other:
- net class Default removed
